File: RX23W/Jan 2020/_autosave-RX23W.sch (KiCad schematic (older format))
At the start: 34 parts, among them SW1 SW_Push, U1 L78L33_SO8, U2 USBLC6-2SC6, U3 RX23W, Y1 54MHz

Commit message: finishing squematic
Parts:
- removed R?: 100, symbol Device:R_Small_US
- added C? (x2): 12pF, symbol Device:C_Small
- added JP?: Jumper_3_Bridged12, symbol Jumper:Jumper_3_Bridged12
- added R?: 10K, symbol Device:R_Small_US
- added R?: 100, symbol Device:R_Small_US
- R?: value 100 -> 4.7K
- R?: value 100 -> 10K
- Y1: value 54MHz -> 16MHz
Connections:
- net GND: now also C?.2, C?.2, R?.1
- net VCC: now also R?.2
- net at U3.23 (PC7): now also JP?.2 (C)
- net at U3.37 (XTAL2_RF), Y?.4: now also C?.1
- net at U3.38 (XTAL1_RF), Y?.1: now also C?.1
- new net: JP?.1 (A), R?.2
- new net: JP?.3 (B), R?.1
Changed lines of the file:
@@
 Wire Wire Line
 	3750 7750 3750 8850
-Text Label 6900 4750 1    50   ~ 0
-3.3V
 $Comp
 L power:VCC #PWR017
@@
 P 5000 2750
 F 0 "Y1" V 4954 3112 50  0000 L CNN
-F 1 "54MHz" V 5045 3112 50  0000 L CNN
+F 1 "16MHz" V 5045 3112 50  0000 L CNN
 F 2 "" H 5000 2750 50  0001 C CNN
 F 3 "~" H 5000 2750 50  0001 C CNN
@@
 Wire Wire Line
 	5250 2450 5250 2200
-Text Label 7600 4900 1    50   ~ 0
-3.3V
-Wire Wire Line
-	7500 4650 7550 4650
 $Comp
 L Jumper:Jumper_3_Bridged12 JP?
@@
 P 5650 1400
 F 0 "R?" V 5521 1446 50  0000 C CNN
-F 1 "100" V 5758 1434 50  0000 C CNN
+F 1 "4.7K" V 5758 1434 50  0000 C CNN
 F 2 "" H 5650 1400 50  0001 C CNN
 F 3 "~" H 5650 1400 50  0001 C CNN
@@
 Wire Wire Line
 	8100 2550 8650 2550
-$Comp
-L Device:R_Small_US R?
-U 1 1 5E8F0AAF
-P 7400 4650
-F 0 "R?" V 7271 4696 50  0000 C CNN
-F 1 "100" V 7508 4684 50  0000 C CNN
-F 2 "" H 7400 4650 50  0001 C CNN
-F 3 "~" H 7400 4650 50  0001 C CNN
-	1    7400 4650
-	0    -1   -1   0
-$EndComp
-$Comp
-L power:VCC #PWR?
-U 1 1 5E886BDA
-P 7550 4650
-F 0 "#PWR?" H 7550 4500 50  0001 C CNN
-F 1 "VCC" H 7567 4823 50  0000 C CNN
-F 2 "" H 7550 4650 50  0001 C CNN
-F 3 "" H 7550 4650 50  0001 C CNN
-	1    7550 4650
-	0    1    1    0
-$EndComp
 Wire Wire Line
 	7300 4650 7200 4650
@@
 P 5250 3350
 F 0 "R?" V 5121 3396 50  0000 C CNN
-F 1 "100" V 5358 3384 50  0000 C CNN
+F 1 "10K" V 5358 3384 50  0000 C CNN
 F 2 "" H 5250 3350 50  0001 C CNN
 F 3 "~" H 5250 3350 50  0001 C CNN
@@
 Wire Notes Line
 	550  4900 550  7700
+$Comp
+L Device:C_Small C?
+U 1 1 5EB66F99
+P 10150 2500
+F 0 "C?" V 10361 2546 50  0000 L CNN
+F 1 "12pF" V 10282 2455 50  0000 L CNN
+F 2 "" H 10150 2500 50  0001 C CNN
+F 3 "~" H 10150 2500 50  0001 C CNN
+	1    10150 2500
+	0    -1   -1   0
+$EndComp
+$Comp
+L Device:C_Small C?
+U 1 1 5EB67AE2
+P 10150 2950
+F 0 "C?" V 10361 2996 50  0000 L CNN
+F 1 "12pF" V 10282 2905 50  0000 L CNN
+F 2 "" H 10150 2950 50  0001 C CNN
+F 3 "~" H 10150 2950 50  0001 C CNN
+	1    10150 2950
+	0    -1   -1   0
+$EndComp
+Wire Wire Line
+	9350 2550 10050 2550
+Wire Wire Line
+	10050 2550 10050 2500
+Connection ~ 9350 2550
+Wire Wire Line
+	10050 2950 9350 2950
+Wire Wire Line
+	9350 2950 9350 2900
+Connection ~ 9350 2900
+Wire Wire Line
+	10250 2950 10250 2750
+$Comp
+L power:GND #PWR?
+U 1 1 5EB8CF01
+P 10400 2750
+F 0 "#PWR?" H 10400 2500 50  0001 C CNN
+F 1 "GND" H 10405 2577 50  0000 C CNN
+F 2 "" H 10400 2750 50  0001 C CNN
+F 3 "" H 10400 2750 50  0001 C CNN
+	1    10400 2750
+	1    0    0    -1
+$EndComp
+Wire Wire Line
+	10400 2750 10250 2750
+Connection ~ 10250 2750
+Wire Wire Line
+	10250 2750 10250 2500
+Wire Wire Line
+	8350 5050 8350 5150
+Wire Wire Line
+	7950 5050 8350 5050
+Wire Wire Line
+	6450 5050 5800 5050
+Wire Wire Line
+	7050 5050 6650 5050
+Wire Wire Line
+	7750 5050 7550 5050
+$Comp
+L Device:R_Small_US R?
+U 1 1 5EBBFE7D
+P 6550 5050
+F 0 "R?" V 6421 5096 50  0000 C CNN
+F 1 "100" V 6658 5084 50  0000 C CNN
+F 2 "" H 6550 5050 50  0001 C CNN
+F 3 "~" H 6550 5050 50  0001 C CNN
+	1    6550 5050
+	0    1    1    0
+$EndComp
+Text Label 5600 5100 0    50   ~ 0
+3.3V
+$Comp
+L Device:R_Small_US R?
+U 1 1 5EBBFE70
+P 7850 5050
+F 0 "R?" V 7721 5096 50  0000 C CNN
+F 1 "10K" V 7958 5084 50  0000 C CNN
+F 2 "" H 7850 5050 50  0001 C CNN
+F 3 "~" H 7850 5050 50  0001 C CNN
+	1    7850 5050
+	0    1    1    0
+$EndComp
+$Comp
+L Jumper:Jumper_3_Bridged12 JP?
+U 1 1 5EBBFE6A
+P 7300 5050
+F 0 "JP?" H 7300 5254 50  0000 C CNN
+F 1 "Jumper_3_Bridged12" H 7300 5163 50  0000 C CNN
+F 2 "" H 7300 5050 50  0001 C CNN
+F 3 "~" H 7300 5050 50  0001 C CNN
+	1    7300 5050
+	-1   0    0    1
+$EndComp
+Text Label 6900 4750 1    50   ~ 0
+3.3V
+Wire Wire Line
+	7300 4650 7300 4900
+$Comp
+L power:GND #PWR?
+U 1 1 5EBF7698
+P 8350 5150
+F 0 "#PWR?" H 8350 4900 50  0001 C CNN
+F 1 "GND" H 8355 4977 50  0000 C CNN
+F 2 "" H 8350 5150 50  0001 C CNN
+F 3 "" H 8350 5150 50  0001 C CNN
+	1    8350 5150
+	1    0    0    -1
+$EndComp
+$Comp
+L power:VCC #PWR?
+U 1 1 5EBFF53E
+P 5800 5050
+F 0 "#PWR?" H 5800 4900 50  0001 C CNN
+F 1 "VCC" H 5818 5223 50  0000 C CNN
+F 2 "" H 5800 5050 50  0001 C CNN
+F 3 "" H 5800 5050 50  0001 C CNN
+	1    5800 5050
+	-1   0    0    1
+$EndComp
 $EndSCHEMATC
