File: RX23W/Jan 2020/RX23W.kicad_pcb (KiCad board)
At the start: 2 copper layers, 39 parts, among them J1 USB_A, SW1 SW_Push, U1 L78L33_SO8, U2 USBLC6-2SC6, U3 RX23W, Y1 16MHz, Y2 32MHz

Commit message: PCB
Routing:
- net GND: vias 50 -> 80
- net (no net): vias 30 -> 0
Changed lines of the file:
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@@
   (gr_line (start 197.9295 99.5045) (end 197.9295 81.28) (layer F.SilkS) (width 0.15))
   (segment (start 178.6975 89.424) (end 178.6975 90.699) (width 0.25) (layer F.Cu) (net 0))
-  (via (at 188.1759 92.1258) (size 0.8) (drill 0.4) (layers F.Cu B.Cu) (net 0))
-  (via (at 187.2234 92.1131) (size 0.8) (drill 0.4) (layers F.Cu B.Cu) (net 0))
-  (via (at 186.2582 92.1131) (size 0.8) (drill 0.4) (layers F.Cu B.Cu) (net 0))
-  (via (at 185.3819 91.9734) (size 0.8) (drill 0.4) (layers F.Cu B.Cu) (net 0))
-  (via (at 189.9539 92.1258) (size 0.8) (drill 0.4) (layers F.Cu B.Cu) (net 0))
-  (via (at 190.8175 92.1131) (size 0.8) (drill 0.4) (layers F.Cu B.Cu) (net 0))
-  (via (at 191.643 91.8083) (size 0.8) (drill 0.4) (layers F.Cu B.Cu) (net 0))
-  (via (at 192.278 91.1987) (size 0.8) (drill 0.4) (layers F.Cu B.Cu) (net 0))
-  (via (at 192.9003 90.551) (size 0.8) (drill 0.4) (layers F.Cu B.Cu) (net 0))
-  (via (at 193.4972 89.9668) (size 0.8) (drill 0.4) (layers F.Cu B.Cu) (net 0))
-  (via (at 194.8815 91.2368) (size 0.8) (drill 0.4) (layers F.Cu B.Cu) (net 0))
-  (via (at 194.2592 91.8464) (size 0.8) (drill 0.4) (layers F.Cu B.Cu) (net 0))
-  (via (at 193.6369 92.456) (size 0.8) (drill 0.4) (layers F.Cu B.Cu) (net 0))
-  (via (at 192.9892 93.1291) (size 0.8) (drill 0.4) (layers F.Cu B.Cu) (net 0))
-  (via (at 192.3669 93.726) (size 0.8) (drill 0.4) (layers F.Cu B.Cu) (net 0))
-  (via (at 191.3128 93.9165) (size 0.8) (drill 0.4) (layers F.Cu B.Cu) (net 0))
-  (via (at 190.3857 93.9165) (size 0.8) (drill 0.4) (layers F.Cu B.Cu) (net 0))
-  (via (at 189.4586 93.9292) (size 0.8) (drill 0.4) (layers F.Cu B.Cu) (net 0))
-  (via (at 188.5315 93.9419) (size 0.8) (drill 0.4) (layers F.Cu B.Cu) (net 0))
-  (via (at 187.5536 93.9292) (size 0.8) (drill 0.4) (layers F.Cu B.Cu) (net 0))
-  (via (at 186.6138 93.9165) (size 0.8) (drill 0.4) (layers F.Cu B.Cu) (net 0))
-  (via (at 185.674 93.9165) (size 0.8) (drill 0.4) (layers F.Cu B.Cu) (net 0))
-  (via (at 184.7215 93.8276) (size 0.8) (drill 0.4) (layers F.Cu B.Cu) (net 0))
-  (via (at 184.0738 93.218) (size 0.8) (drill 0.4) (layers F.Cu B.Cu) (net 0))
-  (via (at 183.3753 92.5322) (size 0.8) (drill 0.4) (layers F.Cu B.Cu) (net 0))
-  (via (at 193.5226 89.027) (size 0.8) (drill 0.4) (layers F.Cu B.Cu) (net 0))
-  (via (at 193.5226 88.011) (size 0.8) (drill 0.4) (layers F.Cu B.Cu) (net 0))
-  (via (at 193.4718 87.0966) (size 0.8) (drill 0.4) (layers F.Cu B.Cu) (net 0))
-  (via (at 195.3895 87.0585) (size 0.7) (drill 0.4) (layers F.Cu B.Cu) (net 0))
-  (via (at 185.7375 82.6135) (size 0.8) (drill 0.4) (layers F.Cu B.Cu) (net 2))
-  (via (at 184.9755 81.5975) (size 0.8) (drill 0.4) (layers F.Cu B.Cu) (net 2))
-  (via (at 187.1345 82.55) (size 0.8) (drill 0.4) (layers F.Cu B.Cu) (net 2))
-  (via (at 188.7855 83.1215) (size 0.8) (drill 0.4) (layers F.Cu B.Cu) (net 2))
-  (via (at 190.119 81.915) (size 0.8) (drill 0.4) (layers F.Cu B.Cu) (net 2))
+  (via (at 188.1759 92.1258) (size 0.8) (drill 0.4) (layers F.Cu B.Cu) (net 2))
+  (via (at 187.2234 92.1131) (size 0.8) (drill 0.4) (layers F.Cu B.Cu) (net 2))
+  (via (at 186.2582 92.1131) (size 0.8) (drill 0.4) (layers F.Cu B.Cu) (net 2))
+  (via (at 185.3819 91.9734) (size 0.8) (drill 0.4) (layers F.Cu B.Cu) (net 2))
+  (via (at 189.9539 92.1258) (size 0.8) (drill 0.4) (layers F.Cu B.Cu) (net 2))
+  (via (at 190.8175 92.1131) (size 0.8) (drill 0.4) (layers F.Cu B.Cu) (net 2))
+  (via (at 191.643 91.8083) (size 0.8) (drill 0.4) (layers F.Cu B.Cu) (net 2))
+  (via (at 192.278 91.1987) (size 0.8) (drill 0.4) (layers F.Cu B.Cu) (net 2))
+  (via (at 192.9003 90.551) (size 0.8) (drill 0.4) (layers F.Cu B.Cu) (net 2))
+  (via (at 193.4972 89.9668) (size 0.8) (drill 0.4) (layers F.Cu B.Cu) (net 2))
+  (via (at 194.8815 91.2368) (size 0.8) (drill 0.4) (layers F.Cu B.Cu) (net 2))
+  (via (at 194.2592 91.8464) (size 0.8) (drill 0.4) (layers F.Cu B.Cu) (net 2))
+  (via (at 193.6369 92.456) (size 0.8) (drill 0.4) (layers F.Cu B.Cu) (net 2))
+  (via (at 192.9892 93.1291) (size 0.8) (drill 0.4) (layers F.Cu B.Cu) (net 2))
+  (via (at 192.3669 93.726) (size 0.8) (drill 0.4) (layers F.Cu B.Cu) (net 2))
+  (via (at 191.3128 93.9165) (size 0.8) (drill 0.4) (layers F.Cu B.Cu) (net 2))
+  (via (at 190.3857 93.9165) (size 0.8) (drill 0.4) (layers F.Cu B.Cu) (net 2))
+  (via (at 189.4586 93.9292) (size 0.8) (drill 0.4) (layers F.Cu B.Cu) (net 2))
+  (via (at 188.5315 93.9419) (size 0.8) (drill 0.4) (layers F.Cu B.Cu) (net 2))
+  (via (at 187.5536 93.9292) (size 0.8) (drill 0.4) (layers F.Cu B.Cu) (net 2))
+  (via (at 186.6138 93.9165) (size 0.8) (drill 0.4) (layers F.Cu B.Cu) (net 2))
+  (via (at 185.674 93.9165) (size 0.8) (drill 0.4) (layers F.Cu B.Cu) (net 2))
+  (via (at 184.7215 93.8276) (size 0.8) (drill 0.4) (layers F.Cu B.Cu) (net 2))
+  (via (at 184.0738 93.218) (size 0.8) (drill 0.4) (layers F.Cu B.Cu) (net 2))
+  (via (at 183.3753 92.5322) (size 0.8) (drill 0.4) (layers F.Cu B.Cu) (net 2))
+  (via (at 193.5226 89.027) (size 0.8) (drill 0.4) (layers F.Cu B.Cu) (net 2))
+  (via (at 193.5226 88.011) (size 0.8) (drill 0.4) (layers F.Cu B.Cu) (net 2))
+  (via (at 193.4718 87.0966) (size 0.8) (drill 0.4) (layers F.Cu B.Cu) (net 2))
+  (via (at 195.3895 87.0585) (size 0.7) (drill 0.4) (layers F.Cu B.Cu) (net 2))
+  (via (at 189.0903 92.1258) (size 0.8) (drill 0.4) (layers F.Cu B.Cu) (net 2))
   (segment (start 150.303 86.318) (end 150.368 86.383) (width 0.25) (layer F.Cu) (net 1))
   (segment (start 150.303 84.709) (end 150.303 86.318) (width 0.25) (layer F.Cu) (net 1))
@@
   (segment (start 144.510001 92.979999) (end 144.15999 93.33001) (width 0.2) (layer F.Cu) (net 1))
   (segment (start 144.15999 93.33001) (end 144.15999 96.298866) (width 0.2) (layer F.Cu) (net 1))
+  (via (at 185.7375 82.6135) (size 0.8) (drill 0.4) (layers F.Cu B.Cu) (net 2))
+  (via (at 184.9755 81.5975) (size 0.8) (drill 0.4) (layers F.Cu B.Cu) (net 2))
+  (via (at 187.1345 82.55) (size 0.8) (drill 0.4) (layers F.Cu B.Cu) (net 2))
+  (via (at 188.7855 83.1215) (size 0.8) (drill 0.4) (layers F.Cu B.Cu) (net 2))
+  (via (at 190.119 81.915) (size 0.8) (drill 0.4) (layers F.Cu B.Cu) (net 2))
   (via (at 172.72 89.408) (size 0.8) (drill 0.4) (layers F.Cu B.Cu) (net 2))
   (via (at 173.99 82.804) (size 0.8) (drill 0.4) (layers F.Cu B.Cu) (net 2))
@@
   (segment (start 171.704 89.3064) (end 171.7548 89.3572) (width 0.2) (layer F.Cu) (net 2))
   (segment (start 171.704 88.092) (end 171.704 89.3064) (width 0.2) (layer F.Cu) (net 2))
-  (via (at 189.0903 92.1258) (size 0.8) (drill 0.4) (layers F.Cu B.Cu) (net 0))
   (via (at 188.976 85.6615) (size 0.8) (drill 0.4) (layers F.Cu B.Cu) (net 2))
   (via (at 187.1345 83.947) (size 0.8) (drill 0.4) (layers F.Cu B.Cu) (net 2))
@@
   )
   (zone (net 2) (net_name GND) (layer F.Cu) (hatch edge 0.508)
+    (priority 1)
     (connect_pads (clearance 0.508))
     (min_thickness 0.254)
-    (fill yes (arc_segments 32) (thermal_gap 0.508) (thermal_bridge_width 0.508))
+    (fill yes (arc_segments 32) (thermal_gap 0.508) (thermal_bridge_width 0.508) (smoothing chamfer) (radius 1))
     (polygon
       (pts

Commit message: PCB 0.2
Parts:
- removed JP1, JP2, JP3: Jumper_3_Bridged12, Button_Switch_SMD:SW_SPDT_PCM12
- added J2: Conn_01x03, Connector_PinHeader_1.00mm:PinHeader_1x03_P1.00mm_Vertical, F.Cu at (91.4, 49.5)
- added J3: Conn_01x03, Connector_PinHeader_1.00mm:PinHeader_1x03_P1.00mm_Vertical, F.Cu at (87.1, 49.5)
- added J4: Conn_01x03, Connector_PinHeader_1.00mm:PinHeader_1x03_P1.00mm_Vertical, F.Cu at (82.8, 49.5)
- C3: footprint Capacitor_SMD:C_0603_1608Metric -> Capacitor_SMD:C_0402_1005Metric
- SW1: footprint Button_Switch_SMD:SW_DIP_SPSTx01_Slide_Copal_CHS-01A_W5.08mm_P1.27mm_JPin -> Button_Switch_SMD:SW_SPST_B3U-3000P-B
- moved R13 117.2 mm to (82.5, 47.8), turned to 0 degrees
- moved R12 105.9 mm to (84.6, 47.8), turned to 0 degrees
- moved Y2 96.0 mm to (94.5, 62.7), turned to 90 degrees
- moved C9 96.0 mm to (93.7, 60.0)
- moved R6 89.1 mm to (94.0, 52.6), turned to 0 degrees
- moved R10 88.6 mm to (87.4, 47.8), turned to 0 degrees
- moved D1 87.2 mm to (91.4, 51.8)
- moved R8 86.6 mm to (115.5, 55.9), turned to 180 degrees
- moved U3 86.4 mm to (99.1, 55.9), turned to 270 degrees
- moved AE1 86.3 mm to (114.9, 49.7)
- moved R9 86.3 mm to (114.8, 54.1)
- moved R7 86.0 mm to (114.8, 57.7)
- moved C13 83.6 mm to (104.9, 59.7), turned to 0 degrees
- moved C12 81.7 mm to (104.9, 58.7), turned to 0 degrees
- moved C6 80.4 mm to (100.8, 49.5)
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Routing:
- net VCC: track 233.9 -> 87.9 mm, vias 0 -> 9
- net USB0_DM: track 44.8 -> 5.63 mm
- net USB0_DP: track 39.6 -> 5.76 mm
- net Net-(J3-Pad2): track 27.3 -> 11.9 mm
- net GND: track 69.2 -> 55.6 mm, vias 80 -> 124
- net VDD: track 19.3 -> 32.7 mm, vias 0 -> 2
- net Net-(J4-Pad2): track 7.53 -> 18.6 mm
- net Net-(R7-Pad1): track 14.8 -> 21.2 mm
- net Net-(C7-Pad2): track 8.66 -> 4.65 mm
- net Net-(J2-Pad2): track 18.7 -> 14.8 mm
- net Net-(U3-Pad37): track 4.27 -> 7.75 mm, vias 0 -> 2
- net Net-(D3-Pad1): track 3.23 -> 0.02 mm
- net Net-(D1-Pad1): track 4.50 -> 1.58 mm
- net Net-(C6-Pad2): track 5.78 -> 8.61 mm
- net Net-(SW1-Pad2): track 7.14 -> 9.54 mm, vias 0 -> 2
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Other:
- board outline added: 44.4 x 18.7 mm
- net class ANT: clearance 0.2 -> 0.1524; via_dia 0.8 -> 0.6; via_drill 0.4 -> 0.3
- net class Default: clearance 0.2 -> 0.1524; trace_width 0.25 -> 0.2; via_dia 0.8 -> 0.6; via_drill 0.4 -> 0.3
- net class GND added: clearance 0.1524, trace_width 0.4, via_dia 0.6, via_drill 0.3
- net class VDD added: clearance 0.1524, trace_width 0.4, via_dia 0.6, via_drill 0.3
- rule trace_clearance: 0.2 -> 0.1524
