File: RX23W/Jan 2020/RX23W.sch (KiCad schematic (older format))
At the start: 26 parts, among them J1 USB_B_Micro, SW1 SW_Push, U1 L78L33_SO8, U2 USBLC6-2SC6, U3 RX23W, Y1 54MHz

Commit message: fishing squematic
Parts:
- removed C2: 10n, symbol Device:C_Small
- removed D4: LED, symbol Device:LED
- removed J1: USB_B_Micro, symbol Connector:USB_B_Micro
- removed R2: 100K, symbol Device:R_Small_US
- added C? (x3): 100nf, symbol Device:C_Small
- added C?: 2.2uF, symbol Device:C_Small
- added D?: LED_CRGB, symbol Device:LED_CRGB
- added J?: USB_A, symbol Connector:USB_A
- added JP?: Jumper_3_Bridged12, symbol Jumper:Jumper_3_Bridged12
- added R? (x4): 100, symbol Device:R_Small_US
- added Y?: 32MHz, symbol Device:Crystal_GND23
Connections:
- net labels removed: ANT, ANTENNA, ARRUMAR, ARRUMARC2, ARRUMARSEP, CLOCK, Circ_1, Circ_2, Circ_3, Circuito1, Circuito2, Circuito3, DCLIN_A, DCLIN_D, ENT_14, ENT_9, FINED, MCU, MCUROTACIONADA1, POWER, RESET, USB, XCOUT
- wire segments 79 -> 142
- no-connect marks 38 -> 26
Other:
- note added: "Circuito de entrada"
- note added: "MCU"
- moved on the sheet: AE1, C1, C10, C3, C5, C6, C7, C8, C9, D3, R1, R4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

Commit message: finishing squematic
Parts:
- removed R?: 100, symbol Device:R_Small_US
- added C? (x2): 12pF, symbol Device:C_Small
- added JP?: Jumper_3_Bridged12, symbol Jumper:Jumper_3_Bridged12
- added R? (x2): 100, symbol Device:R_Small_US
Connections:
- net GND: now also C?.2, C?.2, R?.1
- net VCC: now also R?.2
- net at U3.23 (PC7): now also JP?.2 (C)
- net at U3.37 (XTAL2_RF), Y?.4: now also C?.1
- net at U3.38 (XTAL1_RF), Y?.1: now also C?.1
- new net: JP?.1 (A), R?.2
- new net: JP?.3 (B), R?.1
Changed lines of the file:
@@
 Wire Wire Line
 	3750 7750 3750 8850
-Text Label 6900 4750 1    50   ~ 0
-3.3V
 $Comp
 L power:VCC #PWR017
@@
 Wire Wire Line
 	5250 2450 5250 2200
-Text Label 7600 4900 1    50   ~ 0
-3.3V
-Wire Wire Line
-	7500 4650 7550 4650
 $Comp
 L Jumper:Jumper_3_Bridged12 JP?
@@
 Wire Wire Line
 	8100 2550 8650 2550
-$Comp
-L Device:R_Small_US R?
-U 1 1 5E8F0AAF
-P 7400 4650
-F 0 "R?" V 7271 4696 50  0000 C CNN
-F 1 "100" V 7508 4684 50  0000 C CNN
-F 2 "" H 7400 4650 50  0001 C CNN
-F 3 "~" H 7400 4650 50  0001 C CNN
-	1    7400 4650
-	0    -1   -1   0
-$EndComp
-$Comp
-L power:VCC #PWR?
-U 1 1 5E886BDA
-P 7550 4650
-F 0 "#PWR?" H 7550 4500 50  0001 C CNN
-F 1 "VCC" H 7567 4823 50  0000 C CNN
-F 2 "" H 7550 4650 50  0001 C CNN
-F 3 "" H 7550 4650 50  0001 C CNN
-	1    7550 4650
-	0    1    1    0
-$EndComp
 Wire Wire Line
 	7300 4650 7200 4650
@@
 Wire Notes Line
 	550  4900 550  7700
+$Comp
+L Device:C_Small C?
+U 1 1 5EB66F99
+P 10150 2500
+F 0 "C?" V 10361 2546 50  0000 L CNN
+F 1 "12pF" V 10282 2455 50  0000 L CNN
+F 2 "" H 10150 2500 50  0001 C CNN
+F 3 "~" H 10150 2500 50  0001 C CNN
+	1    10150 2500
+	0    -1   -1   0
+$EndComp
+$Comp
+L Device:C_Small C?
+U 1 1 5EB67AE2
+P 10150 2950
+F 0 "C?" V 10361 2996 50  0000 L CNN
+F 1 "12pF" V 10282 2905 50  0000 L CNN
+F 2 "" H 10150 2950 50  0001 C CNN
+F 3 "~" H 10150 2950 50  0001 C CNN
+	1    10150 2950
+	0    -1   -1   0
+$EndComp
+Wire Wire Line
+	9350 2550 10050 2550
+Wire Wire Line
+	10050 2550 10050 2500
+Connection ~ 9350 2550
+Wire Wire Line
+	10050 2950 9350 2950
+Wire Wire Line
+	9350 2950 9350 2900
+Connection ~ 9350 2900
+Wire Wire Line
+	10250 2950 10250 2750
+$Comp
+L power:GND #PWR?
+U 1 1 5EB8CF01
+P 10400 2750
+F 0 "#PWR?" H 10400 2500 50  0001 C CNN
+F 1 "GND" H 10405 2577 50  0000 C CNN
+F 2 "" H 10400 2750 50  0001 C CNN
+F 3 "" H 10400 2750 50  0001 C CNN
+	1    10400 2750
+	1    0    0    -1
+$EndComp
+Wire Wire Line
+	10400 2750 10250 2750
+Connection ~ 10250 2750
+Wire Wire Line
+	10250 2750 10250 2500
+Wire Wire Line
+	8350 5050 8350 5150
+Wire Wire Line
+	7950 5050 8350 5050
+Wire Wire Line
+	6450 5050 5800 5050
+Wire Wire Line
+	7050 5050 6650 5050
+Wire Wire Line
+	7750 5050 7550 5050
+$Comp
+L Device:R_Small_US R?
+U 1 1 5EBBFE7D
+P 6550 5050
+F 0 "R?" V 6421 5096 50  0000 C CNN
+F 1 "100" V 6658 5084 50  0000 C CNN
+F 2 "" H 6550 5050 50  0001 C CNN
+F 3 "~" H 6550 5050 50  0001 C CNN
+	1    6550 5050
+	0    1    1    0
+$EndComp
+Text Label 5600 5100 0    50   ~ 0
+3.3V
+$Comp
+L Device:R_Small_US R?
+U 1 1 5EBBFE70
+P 7850 5050
+F 0 "R?" V 7721 5096 50  0000 C CNN
+F 1 "100" V 7958 5084 50  0000 C CNN
+F 2 "" H 7850 5050 50  0001 C CNN
+F 3 "~" H 7850 5050 50  0001 C CNN
+	1    7850 5050
+	0    1    1    0
+$EndComp
+$Comp
+L Jumper:Jumper_3_Bridged12 JP?
+U 1 1 5EBBFE6A
+P 7300 5050
+F 0 "JP?" H 7300 5254 50  0000 C CNN
+F 1 "Jumper_3_Bridged12" H 7300 5163 50  0000 C CNN
+F 2 "" H 7300 5050 50  0001 C CNN
+F 3 "~" H 7300 5050 50  0001 C CNN
+	1    7300 5050
+	-1   0    0    1
+$EndComp
+Text Label 6900 4750 1    50   ~ 0
+3.3V
+Wire Wire Line
+	7300 4650 7300 4900
+$Comp
+L power:GND #PWR?
+U 1 1 5EBF7698
+P 8350 5150
+F 0 "#PWR?" H 8350 4900 50  0001 C CNN
+F 1 "GND" H 8355 4977 50  0000 C CNN
+F 2 "" H 8350 5150 50  0001 C CNN
+F 3 "" H 8350 5150 50  0001 C CNN
+	1    8350 5150
+	1    0    0    -1
+$EndComp
+$Comp
+L power:VCC #PWR?
+U 1 1 5EBFF53E
+P 5800 5050
+F 0 "#PWR?" H 5800 4900 50  0001 C CNN
+F 1 "VCC" H 5818 5223 50  0000 C CNN
+F 2 "" H 5800 5050 50  0001 C CNN
+F 3 "" H 5800 5050 50  0001 C CNN
+	1    5800 5050
+	-1   0    0    1
+$EndComp
 $EndSCHEMATC

Commit message: squematic
Parts:
- removed C? (x2): 12pF, symbol Device:C_Small
- removed R?: 100, symbol Device:R_Small_US
- added C2: 1uF, symbol Device:C_Small
- added JP1: Jumper_3_Bridged12, symbol Jumper:Jumper_3_Bridged12
- added R10: 10K, symbol Device:R_Small_US
- added R2: 100, symbol Device:R_Small_US
- R11: renamed from R?; value 100 -> 4.7K
- R13: renamed from R?; value 100 -> 10K
- Y1: value 54MHz -> 16MHz
- gave numbers to parts that had none: 11
Connections:
- net GND: now also C2.2, R10.1
- net VCC: now also U3.16 (P16), R2.2
- net VDD: now also C2.1
- net at U3.10 (P35): now also JP1.2 (C)
- new net: JP1.3 (B), R2.1
- new net: JP1.1 (A), R10.2
- no-connect marks 26 -> 25
Other:
- moved on the sheet: C10, R6

Commit message: squematic
Changed lines of the file:
@@
 	1    0    0    -1
 $EndComp
-Wire Wire Line
-	3750 7750 3750 8850
 $Comp
 L power:VCC #PWR017

Commit message: PCB
Parts:
- removed D1: LED_CRGB, symbol Device:LED_CRGB
- added D1: LED, LED_SMD:LED_0603_1608Metric, symbol Device:LED
- AE1: footprint (none) -> 2450AT42B100E:XCVR_2450AT42B100E
- C1, C10, C11, C12, C13, C2, C4, C5, C6, C7, C8, C9: footprint (none) -> Capacitor_SMD:C_0402_1005Metric
- C3: footprint (none) -> Capacitor_SMD:C_0603_1608Metric
- D3: footprint (none) -> LED_SMD:LED_0603_1608Metric
- J1: footprint (none) -> UJ2-AV-1-SMT:CUI_UJ2-AV-1-SMT
- JP1, JP2, JP3: footprint (none) -> Button_Switch_SMD:SW_SPDT_PCM12
- R1, R10, R11, R12, R13, R2, R3, R4, R5, R6, R8: footprint (none) -> Resistor_SMD:R_0402_1005Metric
- R7, R9: value NC -> 0; footprint (none) -> Resistor_SMD:R_0402_1005Metric
- SW1: footprint (none) -> Button_Switch_SMD:SW_DIP_SPSTx01_Slide_Copal_CHS-01A_W5.08mm_P1.27mm_JPin
- U3: footprint (none) -> Package_DFN_QFN:QFN-56-1EP_7x7mm_P0.4mm_EP5.6x4.6mm_ThermalVias
- Y1, Y2: footprint (none) -> Crystal:Crystal_SMD_2016_2-4Pin_2.0x1.6mm
Connections:
- net GND: no longer R6.1
- net VCC: now also D1.2 (A)
- net at U3.14 (P26): now also R6.2
- new net: D1.1 (K), R6.1
- no-connect marks 25 -> 28
Other:
- moved on the sheet: C10, JP1, R10, R2, R6

Commit message: PCB 0.2
Parts:
- removed JP1, JP2, JP3: Jumper_3_Bridged12, Button_Switch_SMD:SW_SPDT_PCM12, symbol Jumper:Jumper_3_Bridged12
- added J2, J3, J4: Conn_01x03, Connector_PinHeader_1.00mm:PinHeader_1x03_P1.00mm_Vertical, symbol Connector_Generic:Conn_01x03
- C3: footprint Capacitor_SMD:C_0603_1608Metric -> Capacitor_SMD:C_0402_1005Metric
- SW1: footprint Button_Switch_SMD:SW_DIP_SPSTx01_Slide_Copal_CHS-01A_W5.08mm_P1.27mm_JPin -> Button_Switch_SMD:SW_SPST_B3U-3000P-B
Connections:
- net at U3.10 (P35): now also J3.2 (Pin_2)
- net at U3.2 (MD): now also J2.2 (Pin_2)
- net at U3.23 (PC7): now also J4.2 (Pin_2)
- net at R3.2: now also J2.1 (Pin_1)
- net at R11.1: now also J2.3 (Pin_3)
- net at R13.2: now also J4.1 (Pin_1)
- net at R12.1: now also J4.3 (Pin_3)
- net at R2.1: now also J3.3 (Pin_3)
- net at R10.2: now also J3.1 (Pin_1)
Changed lines of the file:
@@
 F 0 "C3" V 8711 1246 50  0000 L CNN
 F 1 "0.47uF" V 8632 1155 50  0000 L CNN
-F 2 "Capacitor_SMD:C_0603_1608Metric" H 8500 1200 50  0001 C CNN
+F 2 "Capacitor_SMD:C_0402_1005Metric" H 8500 1200 50  0001 C CNN
 F 3 "~" H 8500 1200 50  0001 C CNN
 	1    8500 1200
@@
 F 0 "SW1" H 4200 2485 50  0000 C CNN
 F 1 "SW_Push" H 4200 2394 50  0000 C CNN
-F 2 "Button_Switch_SMD:SW_DIP_SPSTx01_Slide_Copal_CHS-01A_W5.08mm_P1.27mm_JPin" H 4200 2400 50  0001 C CNN
+F 2 "Button_Switch_SMD:SW_SPST_B3U-3000P-B" H 4200 2400 50  0001 C CNN
 F 3 "~" H 4200 2400 50  0001 C CNN
 	1    4200 2200
@@
 	5250 2450 5250 2200
 $Comp
-L Jumper:Jumper_3_Bridged12 JP2
-U 1 1 5E88C18C
-P 4900 1400
-F 0 "JP2" H 4900 1604 50  0000 C CNN
-F 1 "Jumper_3_Bridged12" H 4900 1513 50  0000 C CNN
-F 2 "Button_Switch_SMD:SW_SPDT_PCM12" H 4900 1400 50  0001 C CNN
-F 3 "~" H 4900 1400 50  0001 C CNN
-	1    4900 1400
-	1    0    0    -1
-$EndComp
-$Comp
 L Device:R_Small_US R3
 U 1 1 5E89F60E
@@
 $EndComp
 Wire Wire Line
-	4450 1400 4650 1400
-Wire Wire Line
-	5150 1400 5550 1400
-Wire Wire Line
 	5750 1400 6400 1400
 Wire Wire Line
@@
 Wire Wire Line
 	5300 2050 4900 2050
-Wire Wire Line
-	4900 2050 4900 1550
 Wire Wire Line
 	4250 1400 3850 1400
@@
 Wire Wire Line
 	6450 5050 5800 5050
-Wire Wire Line
-	7050 5050 6650 5050
-Wire Wire Line
-	7750 5050 7550 5050
 $Comp
 L Device:R_Small_US R12
@@
 $EndComp
 $Comp
-L Jumper:Jumper_3_Bridged12 JP3
-U 1 1 5EBBFE6A
-P 7300 5050
-F 0 "JP3" H 7300 5254 50  0000 C CNN
-F 1 "Jumper_3_Bridged12" H 7300 5163 50  0000 C CNN
-F 2 "Button_Switch_SMD:SW_SPDT_PCM12" H 7300 5050 50  0001 C CNN
-F 3 "~" H 7300 5050 50  0001 C CNN
-	1    7300 5050
-	-1   0    0    1
-$EndComp
-Wire Wire Line
-	7300 4650 7300 4900
-$Comp
 L power:GND #PWR032
 U 1 1 5EBF7698
@@
 	5950 3250 5950 3400
 Wire Wire Line
-	3800 4050 3600 4050
-Wire Wire Line
 	4700 4050 4900 4050
 $Comp
@@
 	1    4900 4150
 	1    0    0    -1
-$EndComp
-$Comp
-L Jumper:Jumper_3_Bridged12 JP1
-U 1 1 5ED167C2
-P 4050 4050
-F 0 "JP1" H 4050 4254 50  0000 C CNN
-F 1 "Jumper_3_Bridged12" H 4050 4163 50  0000 C CNN
-F 2 "Button_Switch_SMD:SW_SPDT_PCM12" H 4050 4050 50  0001 C CNN
-F 3 "~" H 4050 4050 50  0001 C CNN
-	1    4050 4050
-	-1   0    0    1
 $EndComp
 $Comp
@@
 $EndComp
 Wire Wire Line
-	4500 4050 4300 4050
-Wire Wire Line
 	4900 4050 4900 4150
 Wire Wire Line
@@
 NoConn ~ 6050 3450
 NoConn ~ 6900 3600
+$Comp
+L Connector_Generic:Conn_01x03 J2
+U 1 1 5E46681E
+P 4900 1200
+F 0 "J2" V 4864 1012 50  0000 R CNN
+F 1 "Conn_01x03" V 4773 1012 50  0000 R CNN
+F 2 "Connector_PinHeader_1.00mm:PinHeader_1x03_P1.00mm_Vertical" H 4900 1200 50  0001 C CNN
+F 3 "~" H 4900 1200 50  0001 C CNN
+	1    4900 1200
+	0    -1   -1   0
+$EndComp
+Wire Wire Line
+	5000 1400 5550 1400
+Wire Wire Line
+	4900 1400 4900 2050
+Wire Wire Line
+	4450 1400 4800 1400
+$Comp
+L Connector_Generic:Conn_01x03 J4
+U 1 1 5E4A43D4
+P 7300 5250
+F 0 "J4" V 7172 5430 50  0000 L CNN
+F 1 "Conn_01x03" V 7263 5430 50  0000 L CNN
+F 2 "Connector_PinHeader_1.00mm:PinHeader_1x03_P1.00mm_Vertical" H 7300 5250 50  0001 C CNN
+F 3 "~" H 7300 5250 50  0001 C CNN
+	1    7300 5250
+	0    1    1    0
+$EndComp
+$Comp
+L Connector_Generic:Conn_01x03 J3
+U 1 1 5E4A5268
+P 4050 4250
+F 0 "J3" V 3922 4430 50  0000 L CNN
+F 1 "Conn_01x03" V 4013 4430 50  0000 L CNN
+F 2 "Connector_PinHeader_1.00mm:PinHeader_1x03_P1.00mm_Vertical" H 4050 4250 50  0001 C CNN
+F 3 "~" H 4050 4250 50  0001 C CNN
+	1    4050 4250
+	0    1    1    0
+$EndComp
+Wire Wire Line
+	7300 4650 7300 5050
+Wire Wire Line
+	7400 5050 7750 5050
+Wire Wire Line
+	6650 5050 7200 5050
+Wire Wire Line
+	4050 3900 4050 4050
+Wire Wire Line
+	4150 4050 4500 4050
+Wire Wire Line
+	3600 4050 3950 4050
 $EndSCHEMATC
